File: StepperBreakout.brd (EAGLE design)
At the start: 136.5 x 33.7 mm, 35 parts

Commit message: Improved plane, got rid of cruft
Parts:
- C3: value ECE-V1HA101UP -> EEE-1HA101UP
Routing:
- net VMOT: track 121.6 -> 123.1 mm, vias 0 -> 12
- net VCC: vias 3 -> 2
- added copper zone on layer 16, net VMOT
Other:
- board text added: "100uF EEE-1HA101UP"
- board text removed: "EEE-1HA101UP"
Changed lines of the file:
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@@
 <layer number="27" name="tValues" color="7" fill="1" visible="no" active="yes"/>
 <layer number="28" name="bValues" color="7" fill="1" visible="no" active="yes"/>
-<layer number="29" name="tStop" color="7" fill="3" visible="no" active="yes"/>
-<layer number="30" name="bStop" color="7" fill="6" visible="no" active="yes"/>
+<layer number="29" name="tStop" color="7" fill="3" visible="yes" active="yes"/>
+<layer number="30" name="bStop" color="7" fill="6" visible="yes" active="yes"/>
 <layer number="31" name="tCream" color="7" fill="4" visible="no" active="yes"/>
 <layer number="32" name="bCream" color="7" fill="5" visible="no" active="yes"/>
@@
 <text x="128.905" y="24.13" size="1.27" layer="21" font="vector" ratio="12" rot="R90" align="top-right">A4988 Driver
 Expander</text>
-<text x="38.1" y="31.75" size="1.27" layer="22" font="vector" ratio="12" rot="MR0" align="top-center">EEE-1HA101UP</text>
+<text x="38.1" y="31.75" size="1.27" layer="22" font="vector" ratio="12" rot="MR0" align="top-center">100uF
+EEE-1HA101UP</text>
 </plain>
 <attributes>
@@
 </element>
 <element name="U$7" library="RepRapjr" package="A4988BREAKOUT" value="A4988BREAKOUT" x="3.81" y="7.62" rot="R90"/>
-<element name="C3" library="SparkFun-Capacitors" package="PANASONIC_E" value="ECE-V1HA101UP" x="33.655" y="27.94" rot="R270"/>
+<element name="C3" library="SparkFun-Capacitors" package="PANASONIC_E" value="EEE-1HA101UP" x="33.655" y="27.94" rot="R270"/>
 <element name="C4" library="SparkFun-Capacitors" package="PANASONIC_E" value="" x="42.545" y="27.94" rot="R270"/>
 <element name="C5" library="SparkFun-Capacitors" package="PANASONIC_E" value="" x="42.545" y="17.78" rot="R90"/>
@@
 <contactref element="C5" pad="+"/>
 <contactref element="C6" pad="+"/>
-<wire x1="23.495" y1="15.915" x2="25.44" y2="15.915" width="1.778" layer="1"/>
-<wire x1="25.44" y1="15.915" x2="31.75" y2="22.225" width="1.778" layer="1"/>
-<wire x1="31.75" y1="22.225" x2="33.02" y2="22.225" width="1.778" layer="1"/>
-<wire x1="33.02" y1="22.225" x2="41.91" y2="22.225" width="1.778" layer="1"/>
-<wire x1="41.91" y1="22.225" x2="42.545" y2="22.225" width="1.778" layer="1"/>
-<wire x1="42.545" y1="22.225" x2="46.355" y2="22.225" width="1.778" layer="1"/>
-<wire x1="46.355" y1="22.225" x2="48.26" y2="20.32" width="1.778" layer="1"/>
-<wire x1="42.545" y1="24.94" x2="42.545" y2="22.225" width="1.778" layer="1"/>
+<wire x1="23.495" y1="15.915" x2="26.71" y2="15.915" width="1.778" layer="1"/>
+<wire x1="26.71" y1="15.915" x2="30.48" y2="22.86" width="1.778" layer="1"/>
+<wire x1="30.48" y1="22.86" x2="33.02" y2="22.86" width="1.778" layer="1"/>
+<wire x1="33.655" y1="22.86" x2="41.91" y2="22.86" width="1.778" layer="1"/>
+<wire x1="41.91" y1="22.86" x2="42.545" y2="22.86" width="1.778" layer="1"/>
+<wire x1="42.545" y1="22.86" x2="46.355" y2="22.86" width="1.778" layer="1"/>
+<wire x1="46.355" y1="22.86" x2="48.26" y2="20.32" width="1.778" layer="1"/>
+<wire x1="42.545" y1="24.94" x2="42.545" y2="22.86" width="1.778" layer="1"/>
 <wire x1="33.655" y1="20.78" x2="33.655" y2="21.59" width="1.778" layer="1"/>
-<wire x1="33.655" y1="21.59" x2="33.02" y2="22.225" width="1.778" layer="1"/>
+<wire x1="33.655" y1="21.59" x2="33.02" y2="22.86" width="1.778" layer="1"/>
 <wire x1="33.655" y1="24.94" x2="33.655" y2="22.86" width="1.778" layer="1"/>
-<wire x1="33.655" y1="22.86" x2="33.02" y2="22.225" width="1.778" layer="1"/>
+<wire x1="33.655" y1="22.86" x2="33.02" y2="22.86" width="1.778" layer="1"/>
 <wire x1="42.545" y1="20.78" x2="42.545" y2="21.59" width="1.778" layer="1"/>
-<wire x1="42.545" y1="21.59" x2="41.91" y2="22.225" width="1.778" layer="1"/>
+<wire x1="42.545" y1="21.59" x2="41.91" y2="22.86" width="1.778" layer="1"/>
 <wire x1="41.91" y1="11.037" x2="44.057" y2="11.037" width="0.4064" layer="1"/>
 <wire x1="44.057" y1="11.037" x2="48.26" y2="15.24" width="0.4064" layer="1"/>
+<polygon width="0.6096" layer="16">
+<vertex x="19.05" y="19.05"/>
+<vertex x="19.05" y="29.21" curve="-90"/>
+<vertex x="23.495" y="33.655"/>
+<vertex x="133.35" y="33.655" curve="-90"/>
+<vertex x="137.795" y="29.21"/>
+<vertex x="137.795" y="3.81" curve="-90"/>
+<vertex x="133.985" y="0"/>
+<vertex x="23.495" y="0" curve="-90"/>
+<vertex x="19.05" y="4.445"/>
+</polygon>
+<via x="31.115" y="23.495" extent="1-16" drill="0.5" shape="octagon"/>
+<via x="31.115" y="22.225" extent="1-16" drill="0.5" shape="octagon"/>
+<via x="36.195" y="23.495" extent="1-16" drill="0.5" shape="octagon"/>
+<via x="36.195" y="22.225" extent="1-16" drill="0.5" shape="octagon"/>
+<via x="37.465" y="22.225" extent="1-16" drill="0.5" shape="octagon"/>
+<via x="37.465" y="23.495" extent="1-16" drill="0.5" shape="octagon"/>
+<via x="38.735" y="22.225" extent="1-16" drill="0.5" shape="octagon"/>
+<via x="38.735" y="23.495" extent="1-16" drill="0.5" shape="octagon"/>
+<via x="40.005" y="22.225" extent="1-16" drill="0.5" shape="octagon"/>
+<via x="40.005" y="23.495" extent="1-16" drill="0.5" shape="octagon"/>
+<via x="45.085" y="22.225" extent="1-16" drill="0.5" shape="octagon"/>
+<via x="45.085" y="23.495" extent="1-16" drill="0.5" shape="octagon"/>
 </signal>
 <signal name="N$33">
@@
 <wire x1="46.62" y1="12.33" x2="45.72" y2="11.43" width="0.6096" layer="1"/>
 <wire x1="45.72" y1="11.43" x2="45.72" y2="1.905" width="0.6096" layer="1"/>
-<via x="62.23" y="8.89" extent="1-16" drill="0.6" shape="square"/>
 <wire x1="36.83" y1="6.108" x2="36.83" y2="1.905" width="0.6096" layer="1"/>
 <wire x1="36.83" y1="1.905" x2="26.035" y2="1.905" width="0.8128" layer="1"/>
@@
 <contactref element="U$2" pad="DIR"/>
 <wire x1="66.04" y1="7.62" x2="66.04" y2="5.715" width="0.6096" layer="16"/>
-<wire x1="66.04" y1="5.715" x2="29.845" y2="6.35" width="0.6096" layer="16"/>
 <wire x1="86.36" y1="5.715" x2="66.04" y2="5.715" width="0.6096" layer="16"/>
 <wire x1="86.36" y1="7.62" x2="86.36" y2="5.715" width="0.6096" layer="16"/>
@@
 <wire x1="127" y1="5.715" x2="106.68" y2="5.715" width="0.6096" layer="16"/>
 <contactref element="JP10" pad="5"/>
+<wire x1="66.04" y1="5.715" x2="30.48" y2="5.715" width="0.6096" layer="16"/>
+<wire x1="30.48" y1="5.715" x2="29.845" y2="6.35" width="0.6096" layer="16"/>
 </signal>
 <signal name="EN">
