File: StepperBreakout.sch (EAGLE design)
At the start: 32 parts

Commit message: Improved plane, got rid of cruft
Parts:
- C3: value ECE-V1HA101UP -> EEE-1HA101UP
Changed lines of the file:
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@@
 <part name="JP1" library="SparkFun-Connectors" deviceset="M03X2" device="SHROUD"/>
 <part name="U$7" library="RepRapjr" deviceset="A4988BREAKOUT" device=""/>
-<part name="C3" library="SparkFun-Capacitors" deviceset="CAP_POL" device="E" value="ECE-V1HA101UP"/>
+<part name="C3" library="SparkFun-Capacitors" deviceset="CAP_POL" device="E" value="EEE-1HA101UP"/>
 <part name="C4" library="SparkFun-Capacitors" deviceset="CAP_POL" device="E"/>
 <part name="C5" library="SparkFun-Capacitors" deviceset="CAP_POL" device="E"/>
